File: nanoPhant.sch (EAGLE design)
At the start: 45 parts, among them J1 AMP FCI 10103594-0001LF, U3 ATMEGA32U4, Y1 16MHz

Commit message: Layout done
Parts:
- C1, C10, C2, C3, C4, C5, C6: device SparkFun:CAP0603-CAP -> rcl:C-EUC0603
- J1: device SparkFun-Connectors:USB_MICRO-B_HALF_PTH -> micro usb B - 4LEGS:MICRO-USB-B

Commit message: Routed and Gerber files
Parts:
- LED1: value Red -> Blue
- LED3: value Green -> Red
- R11: value 1K -> 330
- renumbered D1 to LED2, D3 to LED3
Connections:
- removed net N$11: J7.2
- net GND: now also J7.2
Other:
- moved on the sheet: J1
Changed lines of the file:
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@@
 <part name="GND25" library="SparkFun" deviceset="GND" device=""/>
 <part name="GND26" library="SparkFun" deviceset="GND" device=""/>
-<part name="R11" library="SparkFun" deviceset="RESISTOR" device="0603-RES" value="1K"/>
-<part name="LED1" library="SparkFun" deviceset="LED" device="0603" value="Red"/>
+<part name="R11" library="SparkFun" deviceset="RESISTOR" device="0603-RES" value="330"/>
+<part name="LED1" library="SparkFun" deviceset="LED" device="0603" value="Blue"/>
 <part name="GND28" library="SparkFun" deviceset="GND" device=""/>
 <part name="R2" library="SparkFun" deviceset="RESISTOR" device="0603-RES" value="10K"/>
@@
 <part name="GND7" library="SparkFun" deviceset="GND" device=""/>
 <part name="R6" library="SparkFun" deviceset="RESISTOR" device="0603-RES" value="330"/>
-<part name="D3" library="SparkFun" deviceset="LED" device="0603" value="Green"/>
+<part name="LED3" library="SparkFun" deviceset="LED" device="0603" value="Red"/>
 <part name="P+11" library="SparkFun" deviceset="3.3V" device="" value="VCC"/>
 <part name="P+12" library="SparkFun" deviceset="3.3V" device="" value="VCC"/>
@@
 <part name="GND9" library="SparkFun" deviceset="GND" device=""/>
 <part name="R4" library="SparkFun" deviceset="RESISTOR" device="0603-RES" value="330"/>
-<part name="D1" library="SparkFun" deviceset="LED" device="0603" value="Yellow"/>
+<part name="LED2" library="SparkFun" deviceset="LED" device="0603" value="Yellow"/>
 <part name="R5" library="SparkFun" deviceset="RESISTOR" device="0603-RES" value="22"/>
 <part name="R7" library="SparkFun" deviceset="RESISTOR" device="0603-RES" value="22"/>
@@
 <attribute name="VALUE" x="148.082" y="35.306" size="1.524" layer="96"/>
 </instance>
-<instance part="D3" gate="G$1" x="160.02" y="38.1" smashed="yes" rot="R270">
+<instance part="LED3" gate="G$1" x="160.02" y="38.1" smashed="yes" rot="R270">
 <attribute name="NAME" x="163.576" y="40.132" size="1.524" layer="95" rot="R180"/>
 <attribute name="VALUE" x="160.528" y="36.195" size="1.524" layer="96"/>
@@
 <attribute name="VALUE" x="147.828" y="40.386" size="1.524" layer="96"/>
 </instance>
-<instance part="D1" gate="G$1" x="160.02" y="43.18" smashed="yes" rot="R270">
+<instance part="LED2" gate="G$1" x="160.02" y="43.18" smashed="yes" rot="R270">
 <attribute name="NAME" x="163.576" y="45.466" size="1.524" layer="95" rot="R180"/>
 <attribute name="VALUE" x="160.274" y="41.021" size="1.524" layer="96"/>
@@
 <junction x="78.74" y="78.74"/>
 </segment>
+<segment>
+<wire x1="165.1" y1="76.2" x2="165.1" y2="71.12" width="0.1524" layer="91"/>
+<pinref part="GND14" gate="1" pin="GND"/>
+<pinref part="J7" gate="G$1" pin="2"/>
+<wire x1="167.64" y1="76.2" x2="165.1" y2="76.2" width="0.1524" layer="91"/>
+</segment>
 </net>
 <net name="AREF" class="0">
@@
 <segment>
 <pinref part="P+2" gate="1" pin="VCC"/>
-<pinref part="D3" gate="G$1" pin="A"/>
+<pinref part="LED3" gate="G$1" pin="A"/>
 <wire x1="162.56" y1="38.1" x2="167.64" y2="38.1" width="0.1524" layer="91"/>
 <wire x1="167.64" y1="38.1" x2="167.64" y2="43.18" width="0.1524" layer="91"/>
-<pinref part="D1" gate="G$1" pin="A"/>
+<pinref part="LED2" gate="G$1" pin="A"/>
 <wire x1="167.64" y1="43.18" x2="167.64" y2="48.26" width="0.1524" layer="91"/>
 <wire x1="162.56" y1="43.18" x2="167.64" y2="43.18" width="0.1524" layer="91"/>
@@
 <segment>
 <pinref part="R4" gate="G$1" pin="2"/>
-<pinref part="D1" gate="G$1" pin="C"/>
+<pinref part="LED2" gate="G$1" pin="C"/>
 <wire x1="152.4" y1="43.18" x2="154.94" y2="43.18" width="0.1524" layer="91"/>
 </segment>
@@
 <wire x1="154.94" y1="38.1" x2="152.4" y2="38.1" width="0.1524" layer="91"/>
 <pinref part="R6" gate="G$1" pin="2"/>
-<pinref part="D3" gate="G$1" pin="C"/>
+<pinref part="LED3" gate="G$1" pin="C"/>
 </segment>
 </net>
@@
 </segment>
 </net>
-<net name="N$11" class="1">
-<segment>
-<wire x1="167.64" y1="76.2" x2="165.1" y2="76.2" width="0.1524" layer="91"/>
-<wire x1="165.1" y1="76.2" x2="165.1" y2="71.12" width="0.1524" layer="91"/>
-<pinref part="GND14" gate="1" pin="GND"/>
-<pinref part="J7" gate="G$1" pin="2"/>
-</segment>
-</net>

Commit message: Final version
Updated USB footprint, fiducials, images, etc
Parts:
- added FD1, FD2, FD3: FIDUCIAL1X2, SparkFun-Aesthetics:FIDUCIAL1X2
- J1: device micro usb B - 4LEGS:MICRO-USB-B -> pmc_lib:MICRO-USB-B
Connections:
- net GND: now also J7.1, J8.1; no longer J7.2, J8.2
- net VCC: now also J7.2, J8.2; no longer J7.1, J8.1
Changed lines of the file:
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@@
 <part name="F1" library="SparkFun" deviceset="PTC" device="SMD" value="500mA"/>
 <part name="P+2" library="SparkFun" deviceset="VCC" device=""/>
-<part name="J1" library="micro usb B - 4LEGS" deviceset="MICRO-USB-B" device="" value="AMP FCI 10103594-0001LF"/>
+<part name="J1" library="pmc_lib" deviceset="MICRO-USB-B" device="" package3d_urn="urn:adsk.eagle:package:7651683/2" value="AMP FCI 10103594-0001LF"/>
 <part name="FRAME2" library="frames" library_urn="urn:adsk.eagle:library:229" deviceset="A5L-LOC" device=""/>
 <part name="GND5" library="SparkFun" deviceset="GND" device=""/>
@@
 <part name="J7" library="SparkFun-Connectors" deviceset="CONN_04" device=""/>
 <part name="J8" library="SparkFun-Connectors" deviceset="CONN_04" device=""/>
+<part name="FD1" library="SparkFun-Aesthetics" deviceset="FIDUCIAL" device="1X2"/>
+<part name="FD2" library="SparkFun-Aesthetics" deviceset="FIDUCIAL" device="1X2"/>
+<part name="FD3" library="SparkFun-Aesthetics" deviceset="FIDUCIAL" device="1X2"/>
 </parts>
 <sheets>
@@
 <attribute name="VALUE" x="160.274" y="89.662" size="1.524" layer="96"/>
 </instance>
-<instance part="GND18" gate="1" x="144.78" y="111.76" smashed="yes">
-<attribute name="VALUE" x="142.24" y="109.22" size="1.524" layer="96"/>
+<instance part="GND18" gate="1" x="144.78" y="109.22" smashed="yes">
+<attribute name="VALUE" x="142.24" y="106.68" size="1.524" layer="96"/>
 </instance>
 <instance part="P+13" gate="G$1" x="149.86" y="121.92" smashed="yes">
@@
 <attribute name="NAME" x="131.572" y="127" size="1.778" layer="95" font="vector" rot="MR270"/>
 </instance>
+<instance part="FD1" gate="G$1" x="71.12" y="7.62" smashed="yes"/>
+<instance part="FD2" gate="G$1" x="81.28" y="7.62" smashed="yes"/>
+<instance part="FD3" gate="G$1" x="76.2" y="7.62" smashed="yes"/>
 </instances>
 <busses>
@@
 </segment>
 <segment>
-<wire x1="139.7" y1="116.84" x2="139.7" y2="114.3" width="0.1524" layer="91"/>
-<wire x1="139.7" y1="114.3" x2="144.78" y2="114.3" width="0.1524" layer="91"/>
-<pinref part="GND18" gate="1" pin="GND"/>
-<pinref part="J8" gate="G$1" pin="2"/>
-</segment>
-<segment>
 <pinref part="S1" gate="G$1" pin="2"/>
 <pinref part="GND19" gate="1" pin="GND"/>
@@
 </segment>
 <segment>
-<wire x1="165.1" y1="76.2" x2="165.1" y2="71.12" width="0.1524" layer="91"/>
+<pinref part="J7" gate="G$1" pin="1"/>
 <pinref part="GND14" gate="1" pin="GND"/>
-<pinref part="J7" gate="G$1" pin="2"/>
-<wire x1="167.64" y1="76.2" x2="165.1" y2="76.2" width="0.1524" layer="91"/>
+<wire x1="167.64" y1="73.66" x2="165.1" y2="73.66" width="0.1524" layer="91"/>
+<wire x1="165.1" y1="73.66" x2="165.1" y2="71.12" width="0.1524" layer="91"/>
+</segment>
+<segment>
+<pinref part="GND18" gate="1" pin="GND"/>
+<pinref part="J8" gate="G$1" pin="1"/>
+<wire x1="144.78" y1="111.76" x2="144.78" y2="116.84" width="0.1524" layer="91"/>
+<wire x1="144.78" y1="116.84" x2="142.24" y2="116.84" width="0.1524" layer="91"/>
 </segment>
 </net>
@@
 </segment>
 <segment>
-<wire x1="142.24" y1="116.84" x2="149.86" y2="116.84" width="0.1524" layer="91"/>
-<wire x1="149.86" y1="116.84" x2="149.86" y2="121.92" width="0.1524" layer="91"/>
+<wire x1="149.86" y1="114.3" x2="149.86" y2="121.92" width="0.1524" layer="91"/>
 <pinref part="P+13" gate="G$1" pin="3.3V"/>
-<pinref part="J8" gate="G$1" pin="1"/>
+<wire x1="139.7" y1="116.84" x2="139.7" y2="114.3" width="0.1524" layer="91"/>
+<pinref part="J8" gate="G$1" pin="2"/>
+<wire x1="139.7" y1="114.3" x2="149.86" y2="114.3" width="0.1524" layer="91"/>
 </segment>
 <segment>
@@
 </segment>
 <segment>
-<wire x1="167.64" y1="73.66" x2="162.56" y2="73.66" width="0.1524" layer="91"/>
-<wire x1="162.56" y1="73.66" x2="162.56" y2="86.36" width="0.1524" layer="91"/>
+<wire x1="162.56" y1="76.2" x2="162.56" y2="86.36" width="0.1524" layer="91"/>
 <pinref part="P+10" gate="G$1" pin="3.3V"/>
-<pinref part="J7" gate="G$1" pin="1"/>
+<pinref part="J7" gate="G$1" pin="2"/>
+<wire x1="162.56" y1="76.2" x2="167.64" y2="76.2" width="0.1524" layer="91"/>
 </segment>
 </net>
